File: Kicad/BTS-MainBoard-Power.kicad_pcb (KiCad board)
At the start: 2 copper layers, 101.6 x 95.3 mm, 46 parts, among them J1 +12VIn, J10 Conn_01x02, J11 Conn_01x02, J12 Conn_01x02, J13 Conn_01x02, J14 Conn_01x02, J15 Conn_01x02, J16 Conn_01x02, J17 Conn_01x02, J18 Conn_01x02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

Commit message: Renamed Libraries and renamed project files as well
Signed-off-by: bebenlebricolo <benoittarrade@hotmail.fr>
Parts:
- removed U2, U3, U4, U5: STD80N6F6, Package_TO_SOT_SMD:TO-252-2
- added Q1: STD80N6F6, Package_TO_SOT_SMD:TO-252-2, F.Cu at (185.0, 54.6)
- added Q2: STD80N6F6, Package_TO_SOT_SMD:TO-252-2, F.Cu at (183.5, 116.4)
- added Q3: STD80N6F6, Package_TO_SOT_SMD:TO-252-2, F.Cu at (241.5, 53.6)
- added Q4: STD80N6F6, Package_TO_SOT_SMD:TO-252-2, F.Cu at (224.0, 118.5)
- J1, J2: footprint PeltierSwitchingMainBoard:Power_Solder_Pad_7x15mm -> BTS-MainBoard-Power:Power_Solder_Pad_7x15mm
- J10, J11, J4, J5, J6, J7, J8, J9: footprint PeltierSwitchingMainBoard:Power_Solder_Pad_5x10mm_02 -> BTS-MainBoard-Power:Power_Solder_Pad_5x10mm_02
- L1, L2, L3, L4: footprint PeltierSwitchingMainBoard:L_Bourns_SRP1270 -> BTS-MainBoard-Power:L_Bourns_SRP1270
Connections:
- J3 pad 1: Net-(J3-Pad1) -> (no net)
- J3 pad 6: Net-(J3-Pad6) -> (no net)

Commit message: Updated board with FANDRIVE power signal and silkscreen
Signed-off-by: bebenlebricolo <benoittarrade@hotmail.fr>
Parts:
- added REF**: OSHW-Logo2_9.8x8mm_SilkScreen, Symbol:OSHW-Logo2_9.8x8mm_SilkScreen, F.Cu at (208.3, 128.9)
- moved R9 9.16 mm to (215.9, 123.8)
- moved J10 0.13 mm to (229.2, 62.0)
- moved J7 0.13 mm to (229.2, 74.7)
Connections:
- J12 pad 2: GND -> /FanDrive
- J13 pad 2: GND -> /FanDrive
- J14 pad 2: GND -> /FanDrive
- J15 pad 2: GND -> /FanDrive
- J16 pad 2: GND -> /FanDrive
- J17 pad 2: GND -> /FanDrive
- J18 pad 2: GND -> /FanDrive
- J19 pad 2: GND -> /FanDrive
- J3 pad 13: +12V -> /FanDrive
Routing:
- net /FanDrive: track 0.00 -> 175.9 mm
- net GND: track 58.5 -> 11.5 mm
- net /ALS: track 147.7 -> 123.8 mm
- net +12V: track 145.1 -> 161.1 mm
- net /BHS: track 224.4 -> 222.8 mm
- net /BLO: track 94.1 -> 93.4 mm
Other:
- board text added: "+12V"
- board text added: "BTS-MainPower-Control board goes here (mezzanine board)"
- board text added: "Peltier +"
- board text removed: "+12V only"

Commit message: Migrated kicad files to version 6
Signed-off-by: bebenlebricolo <benoittarrade@hotmail.fr>
Other:
- board size 101.6 x 95.3 mm -> 101.6 x 95.2 mm
- net class Default removed
- net class Power track removed
