File: Hardware/V0.2.0/BTS-MainBoard-Power.kicad_sch (KiCad schematic)
At the start: 33 parts, among them J1 +12VIn, J12 Conn_01x02, J13 Conn_01x02, J14 Conn_01x02, J15 Conn_01x02, J16 Conn_01x02, J17 Conn_01x02, J18 Conn_01x02, J19 Conn_01x02, J2 GNDIn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

Commit message: Started first routing steps
Signed-off-by: bebenlebricolo <benoittarrade@hotmail.fr>
Parts:
- removed C?: C_Small, symbol Device:C_Small
- removed J1: +12VIn, BTS-MainBoard-Power:Power_Solder_Pad_7x15mm, symbol Connector_Generic:Conn_01x01
- removed J2: GNDIn, BTS-MainBoard-Power:Power_Solder_Pad_7x15mm, symbol Connector_Generic:Conn_01x01
- added C11: 1uF, Capacitor_SMD:C_1206_3216Metric_Pad1.33x1.80mm_HandSolder, symbol Device:C_Small
- added C12: 100nF, Capacitor_SMD:C_1206_3216Metric_Pad1.33x1.80mm_HandSolder, symbol Device:C_Small
- added D3: 1N4148W, Diode_SMD:D_SOD-123, symbol Diode:1N4148W
- added H5, H6, H7, H8: MountingHole_Pad, MountingHole:MountingHole_3mm_Pad_Via, symbol Mechanical:MountingHole_Pad
- added R10, R11, R12, R9: 220, Resistor_SMD:R_1206_3216Metric_Pad1.30x1.75mm_HandSolder, symbol Device:R
- C7, C9: value C_Small -> 100nF; footprint (none) -> Capacitor_SMD:C_1206_3216Metric_Pad1.33x1.80mm_HandSolder
- C8: value 100nF -> 1uF
- D1, D2: value D_Schottky -> SS56B; footprint (none) -> BTS-MainBoard-Power:SS56B
- H1, H2, H3, H4: footprint MountingHole:MountingHole_4mm_Pad_TopOnly -> MountingHole:MountingHole_4mm_Pad_Via
- J12, J13, J14, J15, J16, J17, J18, J19: value Conn_01x02 -> FanConn; footprint Connector_PinHeader_2.54mm:PinHeader_1x02_P2.54mm_Vertical_SMD_Pin1Left -> Connector_PinSocket_2.54mm:PinSocket_1x02_P2.54mm_Vertical
- J3: value Conn_01x07 -> LogicBoardConnector; footprint (none) -> Connector_PinHeader_2.54mm:PinHeader_1x07_P2.54mm_Vertical
- Q1: value Q_NMOS_DGS -> DMG3418L; footprint (none) -> Package_TO_SOT_SMD:SOT-23
- R2: value 33 -> 1k
Connections:
- net AHO_Sig: now also R10.2
- net ALO_Sig: now also R9.1
- net BHO_Sig: now also R12.2
- net BLO_Sig: now also R11.1
- net FanSink: now also D3.2 (A)
- net GND: now also C11.2, C12.2, H7.1, H8.1, R10.1, R11.2, R12.1, R9.2
- net Psu12V: now also C11.1, C12.1, H5.1, H6.1
- net Vcc: now also D3.1 (K)
- net HBoot2: now reaches C9.1, D2.1 (K), U2.8 (HB)
- net DBootAnode1: now reaches D1.2 (A), R1.1
- net HBoot1: now reaches C7.1, D1.1 (K), U1.8 (HB)
- net DBootAnode2: now reaches D2.2 (A), R3.1
Other:
- note added: "Ground chassis connections"
- note added: "Logic board connection"
- note added: "Mosfet full h bridge implementation"
- note added: "Mosfet half bridge gate drivers"
- note added: "Peltier cooling fans connectors"
- note added: "Peltier cooling fans switching"
- note added: "Power supply connections and filtering"
- note added: "This reverse diode will help to reduce back-emf when switching off cooling fans as they display inductor behaviors"
- note removed: "Peltier fans connectors (40x40mm fans) - No throttling"
- moved on the sheet: C1, C2, C3, C4, C5, C6, C7, C9, D1, H1, H2, H3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

Commit message: Rewired the whole PCB with much more compact design
Signed-off-by: bebenlebricolo <benoittarrade@hotmail.fr>
Parts:
- removed C5: 470uF, Capacitor_SMD:CP_Elec_10x10, symbol Device:C_Polarized
Changed lines of the file:
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@@
   (junction (at 159.385 69.85) (diameter 0) (color 0 0 0 0)
   )
-  (junction (at 60.96 38.735) (diameter 0) (color 0 0 0 0)
-  )
   (junction (at 88.265 93.345) (diameter 0) (color 0 0 0 0)
   )
@@
   (junction (at 175.895 69.85) (diameter 0) (color 0 0 0 0)
   )
-  (junction (at 60.96 31.115) (diameter 0) (color 0 0 0 0)
-  )
   (junction (at 107.315 173.99) (diameter 0) (color 0 0 0 0)
   )
@@
     (stroke (width 0) (type default) (color 0 0 0 0))
   )
-  (wire (pts (xy 60.96 31.115) (xy 69.85 31.115))
-    (stroke (width 0) (type default) (color 0 0 0 0))
-  )
   (wire (pts (xy 147.955 90.17) (xy 157.48 90.17))
     (stroke (width 0) (type default) (color 0 0 0 0))
@@
   )
   (wire (pts (xy 93.98 90.805) (xy 93.98 94.615))
-    (stroke (width 0) (type default) (color 0 0 0 0))
-  )
-  (wire (pts (xy 60.96 38.735) (xy 69.85 38.735))
     (stroke (width 0) (type default) (color 0 0 0 0))
   )
@@
     )
     (property "Datasheet" "~" (id 3) (at 189.23 85.09 0)
-      (effects (font (size 1.27 1.27)) hide)
-    )
-    (pin "1")
-    (pin "2")
-  )
-  (symbol (lib_id "Device:C_Polarized") (at 69.85 34.925 0) (unit 1)
-    (in_bom yes) (on_board yes) (fields_autoplaced)
-    (property "Reference" "C5" (id 0) (at 72.771 33.1275 0)
-      (effects (font (size 1.27 1.27)) (justify left))
-    )
-    (property "Value" "470uF" (id 1) (at 72.771 35.9026 0)
-      (effects (font (size 1.27 1.27)) (justify left))
-    )
-    (property "Footprint" "Capacitor_SMD:CP_Elec_10x10" (id 2) (at 70.8152 38.735 0)
-      (effects (font (size 1.27 1.27)) hide)
-    )
-    (property "Datasheet" "~" (id 3) (at 69.85 34.925 0)
       (effects (font (size 1.27 1.27)) hide)
     )
@@
       (reference "C4") (unit 1) (value "470uF") (footprint "Capacitor_SMD:CP_Elec_10x10")
     )
-    (path "/1c4eb5ab-be48-4ab0-8c07-7bb64a491b21"
-      (reference "C5") (unit 1) (value "470uF") (footprint "Capacitor_SMD:CP_Elec_10x10")
-    )
     (path "/a4fa9b07-ccd0-42a6-99f7-bd04003d6c61"

Commit message: Finished routing, now needs improvements
Signed-off-by: bebenlebricolo <benoittarrade@hotmail.fr>
Connections:
- net Vcc is gone; now on net Psu12V: D3.1 (K), J12.1 (Pin_1), J13.1 (Pin_1), J14.1 (Pin_1), J15.1 (Pin_1), J16.1 (Pin_1), J17.1 (Pin_1), J18.1 (Pin_1), J19.1 (Pin_1)
Changed lines of the file:
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@@
+    (effects (font (size 1.27 1.27)) (justify right bottom))
+  )
+  (label "Psu12V" (at 100.33 128.27 180)
     (effects (font (size 1.27 1.27)) (justify right bottom))
   )
@@
     (effects (font (size 1.27 1.27)) (justify left bottom))
   )
-  (label "Vcc" (at 100.33 128.27 180)
-    (effects (font (size 1.27 1.27)) (justify right bottom))
-  )
   (label "CoolingFanDriveSignal" (at 44.45 80.01 180)

Commit message: Updated the board with logo and silkscreen improvements
Signed-off-by: bebenlebricolo <benoittarrade@hotmail.fr>
Parts:
- added D4: LED, Diode_SMD:D_0805_2012Metric, symbol Device:LED
- added R13: 1k, Resistor_SMD:R_1206_3216Metric_Pad1.30x1.75mm_HandSolder, symbol Device:R
- added TP1, TP13, TP14, TP15, TP16, TP17, TP18, TP19, TP2, TP6, TP7, TP8, TP9: TestPoint, TestPoint:TestPoint_Pad_D1.0mm, symbol Connector:TestPoint
Connections:
- net AHO_Sig: now also TP1.1
- net ALO_Sig: now also TP2.1
- net BHO_Sig: now also TP8.1
- net BLO_Sig: now also TP9.1
- net CoolingFanDriveSignal: now also TP17.1
- net DBootAnode1: now also TP7.1
- net DBootAnode2: now also TP14.1
- net FanSink: now also TP18.1
- net GND: now also D4.1 (K), TP16.1
- net HBoot1: now also TP6.1
- net HBoot2: now also TP13.1
- net Psu12V: now also R13.1, TP15.1
- net VSense: now also TP19.1
- new net: D4.2 (A), R13.2
Other:
- note added: "Gate drivers test points"
- note added: "Other test points"
- moved on the sheet: D3, J12, J13, J14, J15, J16, J17, J18, J19, Q1, R2
